File: KiCAD-Project/b5s4-XA1541-active.kicad_pcb (KiCad board)
At the start: 2 copper layers, 45.6 x 51.8 mm, 10 parts, among them CN1 Male DB25 - Parallel Port, CN2 C64 Serial Connector - DIN 45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, Q1 2N3904, Q2 2N3904, Q3 2N3904, Q4 2N3904

Commit message: Added PDF schematics
Other:
- board text added: "Rev 1.1 - Some additional notes on the silkscreen - Moved some stitching vias - DIN socket was mounted in reverse"
- board text added: "Rev 1.2 - Removed some right angles in the traces - Some minor silkscreen improvements"
- board text removed: "Rev 1.1 - Some additional notes on the silkscreen - Moved some stiching vias - DIN socket was mounted in reverse"
- board text removed: "Rev 1.2 - Removed some right angles in the traces - Additional Via stiching - Some minor Silkscreen improvements"
Changed lines of the file:
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@@
 	(paper "A4")
 	(title_block
-		(title "XA1541-active")
-		(rev "1.1")
+		(title "b5s4 XA1541 active")
+		(rev "1.2")
+		(company "Oddsocks b5s4")
 	)
 	(layers
@@
 			(usegerberattributes yes)
 			(usegerberadvancedattributes yes)
-			(creategerberjobfile no)
+			(creategerberjobfile yes)
 			(dashed_line_dash_ratio 12.000000)
 			(dashed_line_gap_ratio 3.000000)
@@
 			(sketchdnponfab yes)
 			(crossoutdnponfab yes)
-			(subtractmaskfromsilk no)
+			(subtractmaskfromsilk yes)
 			(outputformat 1)
 			(mirror no)
 			(drillshape 0)
 			(scaleselection 1)
-			(outputdirectory "pcbway-gerbers")
+			(outputdirectory "gerbers")
 		)
 	)
@@
 		)
 	)
-	(gr_text "Rev 1.2\n- Removed some right angles in the traces\n- Additional Via stiching\n- Some minor Silkscreen improvements\n"
+	(gr_text "Rev 1.2\n- Removed some right angles in the traces\n- Some minor silkscreen improvements\n"
 		(at 149.86 81.28 0)
 		(layer "User.1")
@@
 		)
 	)
-	(gr_text "Rev 1.1\n- Some additional notes on the silkscreen\n- Moved some stiching vias\n- DIN socket was mounted in reverse\n"
+	(gr_text "Rev 1.1\n- Some additional notes on the silkscreen\n- Moved some stitching vias\n- DIN socket was mounted in reverse\n"
 		(at 149.86 73.66 0)
 		(layer "User.1")
