File: KiCAD-Project/b5s4-XA1541-active.kicad_sch (KiCad schematic)
At the start: 10 parts, among them CN1 Male DB25 - Parallel Port, CN2 C64 Serial Connector - DIN 45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, Q1 2N3904, Q2 2N3904, Q3 2N3904, Q4 2N3904

Commit message: Added PDF schematics
Other:
- note added: "Original circuit design is © by Michael Klein and Nicolas Welte, 2000."
- company: (none) -> Oddsocks b5s4
- title: XA1541-active -> b5s4 XA1541 active
Changed lines of the file:
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@@
 	(paper "A4")
 	(title_block
-		(title "XA1541-active")
+		(title "b5s4 XA1541 active")
+		(rev "1.2")
+		(company "Oddsocks b5s4")
+	)
+	(text "Original circuit design is © by Michael Klein and Nicolas Welte, 2000."
+		(exclude_from_sim no)
+		(at 151.384 145.796 0)
+		(effects
+			(font
+				(size 1.27 1.27)
+			)
+		)
 	)
 	(junction
